File: hardware/astracompanion/astracompanion.kicad_sch (KiCad schematic)
At the start: 102 parts, among them J1 Screw_Terminal_01x02, J10 Conn_01x03_Pin, J2 Screw_Terminal_01x02, J3 Conn_01x03_Pin, J4 USB_C_Receptacle_USB2.0, J5 Conn_01x02_Socket, J6 Micro_SD_Card, J7 Conn_01x04_Socket, J8 testpoint, J9 Encoder_L, Q4 AO3401A, SW1 PTS645, SW2 SW_SPST, SW3 PTS645, SW4 Reset / EN button, SW5 Boot / IO0 button, SW6 PTS645, U1 MT3608_BOOSTER_MODULE, U10 MAX17048G+T10, U11 USBLC6-2SC6, U13 USBLC6-4SC6, U2 ESP32-S3-DEVKITC-1-N8R8, U3 DRV8833PWP, U4 MAX98357A, U5 MPU-6050, U6 DS3231M, U7 AP2112K-3.3, U8 VL53L0CXV0DH1

Commit message: Add firmware skeleton and document the current hardware
Co-authored-by: Cursor <cursoragent@cursor.com>
Parts:
- BT1: footprint Battery:BatteryHolder_Keystone_1042_1x18650 -> Connector_JST:JST_PH_B2B-PH-K_1x02_P2.00mm_Vertical
Changed lines of the file:
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@@
 			)
 		)
-		(property "Footprint" "Battery:BatteryHolder_Keystone_1042_1x18650"
+		(property "Footprint" "Connector_JST:JST_PH_B2B-PH-K_1x02_P2.00mm_Vertical"
 			(at 93.98 74.676 90)
 			(hide yes)

Commit message: Ship the laptop voice stack, Phase 6 robot contract, and ESP32 firmware.
Local secrets, config, and databases stay gitignored.

Co-authored-by: Cursor <cursoragent@cursor.com>
Parts:
- removed U2: ESP32-S3-DEVKITC-1-N8R8, Connector_PinHeader_2.54mm:PinHeader_2x19_P2.54mm_Vertical, symbol ESP32-S3-DEVKITC-1-N8R8:ESP32-S3-DEVKITC-1-N8R8
- added U17, UE1: Conn_01x22_Pin, Connector_PinSocket_2.54mm:PinSocket_1x22_P2.54mm_Vertical, symbol Connector:Conn_01x22_Pin
Connections:
- net BTN_SELECT: now also U17.5 (Pin_5)
- net BTN_UP: now also U17.4 (Pin_4)
- net GND: now also U17.1 (Pin_1), U17.21 (Pin_21), U17.22 (Pin_22)
- net I2S_BCLK: now also U17.15 (Pin_15)
- net I2S_DOUT: now also U17.2 (Pin_2)
- net I2S_LRCK: now also U17.16 (Pin_16)
- net MOTOR_L_DIR: now also U17.8 (Pin_8)
- net MOTOR_L_PWM: now also U17.9 (Pin_9)
- net MOTOR_R_DIR: now also U17.6 (Pin_6)
- net MOTOR_R_PWM: now also U17.7 (Pin_7)
- net RGB_DATA: now also U17.10 (Pin_10)
- net SD_CS: now also U17.18 (Pin_18)
- net SPI_MISO: now also U17.17 (Pin_17)
- net USB_D+: now also U17.19 (Pin_19)
- net USB_D-: now also U17.20 (Pin_20)
- net at R16.2, SW5.1: now also U17.14 (Pin_14)
